File: LedMatrix.kicad_sch (KiCad schematic)
At the start: 13 parts, among them J1 External Pwr, U1 MAX7219, U2 TDCR1060M, U3 TDCR1060M

Commit message: Completed LED 7-Segment Board
Parts:
- added H1, H2, H3: MountingHole_Pad, MountingHole:MountingHole_3.2mm_M3_DIN965_Pad, symbol Mechanical:MountingHole_Pad
- added LS1: Buzzer, LedMatrixFootprintLib:Buzzer, symbol New_Library:AT-1224-TWT-5V-2-R
- C1: footprint (none) -> Capacitor_SMD:C_0805_2012Metric_Pad1.18x1.45mm_HandSolder
- C2: footprint (none) -> LedMatrixFootprintLib:CAP_YX_5X11_RUB
- D1: footprint (none) -> Diode_SMD:D_0805_2012Metric_Pad1.15x1.40mm_HandSolder
- J1: footprint (none) -> Connector_PinHeader_2.54mm:PinHeader_1x02_P2.54mm_Vertical
- R1, R2: footprint (none) -> Resistor_SMD:R_1206_3216Metric_Pad1.30x1.75mm_HandSolder
- S1: renamed from S2; value Button2 -> Mode; footprint VS-1213-67-160GF:SW_VS-1213-67-160GF -> LedMatrixFootprintLib:SW_VS-1213-67-160GF
- S2: renamed from S1; value Button1 -> Reset; footprint VS-1213-67-160GF:SW_VS-1213-67-160GF -> LedMatrixFootprintLib:SW_VS-1213-67-160GF
- S3: value Button3 -> Start/Stop; footprint VS-1213-67-160GF:SW_VS-1213-67-160GF -> LedMatrixFootprintLib:SW_VS-1213-67-160GF
- U1: footprint (none) -> LedMatrixFootprintLib:21-0043D_24_MXM
- U2, U3: footprint TDCG1060M_VIS -> LedMatrixFootprintLib:TDCG1060M_VIS
Connections:
- net GND: now also H1.1, H2.1, H3.1, LS1.N
- net Mode: now also A1.6 (D3), S1.1, S1.2; no longer A1.5 (D2), S2.1, S2.2
- net Reset: now also A1.5 (D2), S2.1, S2.2; no longer A1.6 (D3), S1.1, S1.2
- net Buzzer: now reaches A1.12 (D9)
- net Buzzer: now also LS1.P
Other:
- moved on the sheet: S1, S2
